File: pca-electronics/pca-electronics.kicad_sch (KiCad schematic)
At the start: 0 parts

Commit message: Rough initial prototype work
Parts:
- added A1: Adafruit_Feather_Generic, Module:Adafruit_Feather, symbol MCU_Module:Adafruit_Feather_Generic
- added J1, J2, J3, J4: 12V Out, Connector_AMASS:AMASS_XT30U-M_1x02_P5.0mm_Vertical, symbol Connector_Generic:Conn_01x02
- added J5, J6, J7, J8: 10k Analog Read, Connector_JST:JST_PH_B2B-PH-K_1x02_P2.00mm_Vertical, symbol Connector_Generic:Conn_01x02
- added J9: 12V In, Connector_AMASS:AMASS_XT30U-F_1x02_P5.0mm_Vertical, symbol Connector_Generic:Conn_01x02
- added Q1, Q2, Q3, Q4: IRLB8721PBF, Package_TO_SOT_THT:TO-220-3_Vertical, symbol Transistor_FET:IRLB8721PBF
- added R1, R2, R3, R4: R_US, Resistor_THT:R_Axial_DIN0204_L3.6mm_D1.6mm_P7.62mm_Horizontal, symbol Device:R_US
Connections:
- new net: J2.1 (Pin_1), Q2.2 (D)
- new net: J4.1 (Pin_1), Q4.2 (D)
- new net: J3.1 (Pin_1), Q3.2 (D)
- new net: J1.1 (Pin_1), Q1.2 (D)
- new net +12V: J1.2 (Pin_2), J2.2 (Pin_2), J3.2 (Pin_2), J4.2 (Pin_2), J9.1 (12_V_in)
- new net 3V3: A1.2 (3V3), J5.2 (Pin_2), J6.2 (Pin_2), J7.2 (Pin_2), J8.2 (Pin_2)
- new net A0: A1.5 (A0), J5.1 (Pin_1), R1.1
- new net A1: A1.6 (A1), J6.1 (Pin_1), R2.1
- new net A2: A1.7 (A2), J7.1 (Pin_1), R3.1
- new net A3: A1.8 (A3), J8.1 (Pin_1), R4.1
- new net A4: A1.9 (A4)
- new net A5: A1.10 (A5)
- new net AREF: A1.3 (AREF)
- new net D0: A1.19 (D0), Q4.1 (G)
- new net D1: A1.20 (D1)
- new net D2: A1.21 (D2)
- new net D3: A1.22 (D3)
- new net D4: A1.23 (D4), Q2.1 (G)
- new net D5: A1.24 (D5), Q1.1 (G)
- new net D6: A1.25 (D6), Q3.1 (G)
- new net EN: A1.27 (EN)
- new net GND: A1.4 (GND), J9.2 (GND), Q1.3 (S), Q2.3 (S), Q3.3 (S), Q4.3 (S), R1.2, R2.2, R3.2, R4.2
- new net MISO: A1.13 (MISO)
- new net MOSI: A1.12 (MOSI)
- new net RESET: A1.1 (~{RESET})
- new net RX: A1.14 (RX)
- new net SCK: A1.11 (SCK)
- new net SCL: A1.18 (SCL)
- new net SDA: A1.17 (SDA)
- new net SPARE: A1.16 (SPARE)
- new net TX: A1.15 (TX)
- new net USB: A1.26 (USB)
- new net VBAT: A1.28 (VBAT)
